Commit message: Drawing robot description and gazebo: Gazebo config for base simulation ready

File: drawing_robot_description/urdf/colors_and_materials.xacro (robot description, xacro)
@@ -1,4 +1,4 @@
 <robot name="xacro_properties" xmlns:xacro="http://ros.org/wiki/xacro">
-    <material name="gray_pla">
+    <material name="grey_pla">
         <color rgba="0.552 0.501 0.501 1"/>
     </material>

File: drawing_robot_description/urdf/drawing_robot_description.urdf.xacro (robot description, xacro)
@@ -3,4 +3,5 @@
   <!-- ____________________________________ XACRO IMPORTS AND PROPERTIES _______________________________________-->
   <xacro:include filename="$(find drawing_robot_description)/urdf/colors_and_materials.xacro"/>
+  <xacro:include filename="$(find drawing_robot_description)/urdf/drawing_robot_gazebo.urdf.xacro"/>
   <xacro:property name="angle_servo" value="1.5707" />
   <xacro:property name="black_servo" value="7.605" />
@@ -32,5 +33,5 @@
           filename="package://drawing_robot_description/meshes/base_link.STL" />
       </geometry>
-      <material name="gray_pla"/>
+      <material name="grey_pla"/>
     </visual>
     <collision>
@@ -69,5 +70,5 @@
           filename="package://drawing_robot_description/meshes/arm_1.STL" />
       </geometry>
-      <material name="gray_pla"/>
+      <material name="grey_pla"/>
     </visual>
     <collision>
@@ -124,5 +125,5 @@
           filename="package://drawing_robot_description/meshes/arm_2.STL" />
       </geometry>
-      <material name="gray_pla"/>
+      <material name="grey_pla"/>
     </visual>
     <collision>
