Commit message: Drawing robot description and gazebo: Adding controllers and transmission, some configs are still missing

File: drawing_robot_description/urdf/drawing_robot_description.urdf.xacro (robot description, xacro)
@@ -4,4 +4,5 @@
   <xacro:include filename="$(find drawing_robot_description)/urdf/colors_and_materials.xacro"/>
   <xacro:include filename="$(find drawing_robot_description)/urdf/drawing_robot_gazebo.urdf.xacro"/>
+  <xacro:include filename="$(find drawing_robot_description)/urdf/drawing_robot_transmission.urdf.xacro"/>
   <xacro:property name="angle_servo" value="1.5707" />
   <xacro:property name="black_servo" value="7.605" />
@@ -9,4 +10,10 @@
   <xacro:property name="offset_pen" value="-0.02" />
   <!-- ____________________________________ BASE LINK DEFINITIONS ______________________________________________-->
+  <link name="world"/>
+  <joint name="base_joint" type="fixed">
+    <parent link="world"/>
+    <child link="base_link"/>
+    <origin xyz="0.0 0.0 0.0175"/>
+  </joint>
   <link
     name="base_link">
@@ -100,5 +107,5 @@
       velocity="8.05" />
   </joint>
-  <!-- ________________________________________ ARM 1 DEFINITIONS ______________________________________________-->
+  <!-- ________________________________________ ARM 2 DEFINITIONS ______________________________________________-->
   <link
     name="arm_2">
@@ -155,5 +162,5 @@
       velocity="8.05" />
   </joint>
-  <!-- ________________________________________ ARM 2 DEFINITIONS ______________________________________________-->
+  <!-- ________________________________________ END EFFECTOR DEFINITIONS ______________________________________________-->
   <link
     name="hand">

File: drawing_robot_description/urdf/drawing_robot_gazebo.urdf.xacro (robot description, xacro)
@@ -3,16 +3,20 @@
     reference="base_link">
     <material>Gazebo/Grey</material>
+    <selfCollide>true</selfCollide>
   </gazebo>
   <gazebo
     reference="arm_1">
     <material>Gazebo/Grey</material>
+    <selfCollide>true</selfCollide>
   </gazebo>
   <gazebo
     reference="arm_2">
     <material>Gazebo/Grey</material>
+    <selfCollide>true</selfCollide>
   </gazebo>
   <gazebo
     reference="hand">
     <material>Gazebo/SkyBlue</material>
+    <selfCollide>true</selfCollide>
   </gazebo>
 </robot>
