Commit message: Ezzybot MK2 Description: Mounted bse of the robot

File: eezybot_mk2_description/urdf/mk2_base.urdf.xacro (robot description, xacro)
@@ -1,36 +1,218 @@
 <?xml version="1.0"?>
 <robot xmlns:xacro="http://www.ros.org/wiki/xacro">
-    <xacro:macro name="spacer_m4x17"
-            params="id parent  x y z">
-        <!-- Link -->
-        <link name="${id}">
-        <visual>
-            <origin xyz="0 0 0" rpy="0 0 0"/>
-            <geometry>
-            <mesh filename="package://eezybot_mk2_description/meshes/spacer_m4x17.stl"
-                scale="0.001 0.001 0.001"/>
-            </geometry>
-            <material name="SoftBlack"/>
-        </visual>
-        <collision>
-            <origin xyz="0 0 0" rpy="0 0 0"/>
-            <geometry>
-            <mesh filename="package://eezybot_mk2_description/meshes/spacer_m4x17.stl"
-                scale="0.001 0.001 0.001"/>
-            </geometry>
-        </collision>
-        <inertial>
-            <origin xyz="0 0 0"/>
-            <mass value="0.0053"/>
-            <inertia ixx="0.001" ixy="0.0" ixz="0.0"
-                    iyy="0.001" iyz="0.0"
-                    izz="0.001"/>
-        </inertial>
-        </link>
-        <joint name="${id}_joint" type="fixed">
-        <parent link="${parent}"/>
-        <child link="${id}_${element}"/>
-        <origin xyz="${x} ${y} ${z}" rpy="0 0 0"/>
-        </joint>
-    </xacro:macro>
+    <link name="base_link" />
+    <link name="main_base">
+    <visual>
+        <origin xyz="-0.041 -0.0444 0" rpy="0 0 0"/>
+        <geometry>
+        <mesh filename="package://eezybot_mk2_description/meshes/EBAmk2_012_mainbase.STL"
+            scale="0.001 0.001 0.001"/>
+        </geometry>
+        <material name="OrangePLA"/>
+    </visual>
+    <collision>
+        <origin xyz="-0.041 -0.0444 0" rpy="0 0 0"/>
+        <geometry>
+        <mesh filename="package://eezybot_mk2_description/meshes/EBAmk2_012_mainbase.STL"
+            scale="0.001 0.001 0.001"/>
+        </geometry>
+    </collision>
+    <inertial>
+        <origin xyz="0 0 0"/>
+        <mass value="0.0053"/>
+        <inertia ixx="0.001" ixy="0.0" ixz="0.0"
+                iyy="0.001" iyz="0.0"
+                izz="0.001"/>
+    </inertial>
+    </link>
+    <joint name="main_base_joint" type="fixed">
+        <parent link="base_link"/>
+        <child link="main_base"/>
+        <origin xyz="0 0 0" rpy="0 0 0"/>
+    </joint>
+    <link name="MG996r_1">
+    <visual>
+        <origin xyz="0 0 0" rpy="0 0 0"/>
+        <geometry>
+        <mesh filename="package://eezybot_mk2_description/meshes/MG946R-MG946R.stl"
+            scale="1 1 1"/>
+        </geometry>
+        <material name="BlackPLA"/>
+    </visual>
+    <collision>
+        <origin xyz="0 0 0" rpy="0 0 0"/>
+        <geometry>
+        <mesh filename="package://eezybot_mk2_description/meshes/MG946R-MG946R.stl"
+            scale="1 1 1"/>
+        </geometry>
+    </collision>
+    <inertial>
+        <origin xyz="0 0 0"/>
+        <mass value="0.0053"/>
+        <inertia ixx="0.001" ixy="0.0" ixz="0.0"
+                iyy="0.001" iyz="0.0"
+                izz="0.001"/>
+    </inertial>
+    </link>
+    <joint name="MG996r_1_joint" type="fixed">
+        <parent link="main_base"/>
+        <child link="MG996r_1"/>
+        <origin xyz="-0.0075 0.001 0.008" rpy="0 0 0"/>
+    </joint>
+    <link name="MG996r_conn1">
+    <visual>
+        <origin xyz="0 0 0" rpy="0 0 0"/>
+        <geometry>
+        <mesh filename="package://eezybot_mk2_description/meshes/MG946R_piattelo-MG946R_piattelo.stl"
+            scale="1 1 1"/>
+        </geometry>
+        <material name="BlackPLA"/>
+    </visual>
+    <collision>
+        <origin xyz="0 0 0" rpy="0 0 0"/>
+        <geometry>
+        <mesh filename="package://eezybot_mk2_description/meshes/MG946R_piattelo-MG946R_piattelo.stl"
+            scale="1 1 1"/>
+        </geometry>
+    </collision>
+    <inertial>
+        <origin xyz="0 0 0"/>
+        <mass value="0.0053"/>
+        <inertia ixx="0.001" ixy="0.0" ixz="0.0"
+                iyy="0.001" iyz="0.0"
+                izz="0.001"/>
+    </inertial>
+    </link>
+    <joint name="MG996r_conn1_joint" type="revolute">
+        <parent link="MG996r_1"/>
+        <child link="MG996r_conn1"/>
+        <origin xyz="0.01 0 0.0385" rpy="0 0 0"/>
+        <axis xyz="0.0 0.0 1.0"/>
+        <limit lower="-1.57" upper="1.57" effort="5.0" velocity="1.0"/>
+        <dynamics damping="0.1" friction="0.01"/>
+        <safety_controller soft_lower_limit="-1.4" soft_upper_limit="1.4" k_position="10" k_velocity="5"/>
+        <calibration rising="0.0" falling="0.0"/>
+    </joint>
+    <link name="gearservo_1">
+    <visual>
+        <origin xyz="${-0.012935 * 1.575} ${0.012935 * 1.575} 0" rpy="${pi} 0 0"/>
+        <geometry>
+        <mesh filename="package://eezybot_mk2_description/meshes/EBAmk2_010_gearservo.STL"
+            scale="0.001 0.001 0.001"/>
+        </geometry>
+        <material name="OrangePLA"/>
+    </visual>
+    <collision>
+        <origin xyz="${-0.012935 * 1.575} ${0.012935 * 1.575} 0" rpy="${pi} 0 0"/>
+        <geometry>
+        <mesh filename="package://eezybot_mk2_description/meshes/EBAmk2_010_gearservo.STL"
+            scale="0.001 0.001 0.001"/>
+        </geometry>
+    </collision>
+    <inertial>
+        <origin xyz="0 0 0"/>
+        <mass value="0.0053"/>
+        <inertia ixx="0.001" ixy="0.0" ixz="0.0"
+                iyy="0.001" iyz="0.0"
+                izz="0.001"/>
+    </inertial>
+    </link>
+    <joint name="gearservo_1joint" type="fixed">
+        <parent link="MG996r_conn1"/>
+        <child link="gearservo_1"/>
+        <origin xyz="0 0 0.0025" rpy="0 0 0"/>
+    </joint>
+    <link name="lower_base">
+    <visual>
+        <origin xyz="-0.0455 -0.0415 0" rpy="0 0 0"/>
+        <geometry>
+        <mesh filename="package://eezybot_mk2_description/meshes/EBAmk2_013_lower_base.STL"
+            scale="0.001 0.001 0.001"/>
+        </geometry>
+        <material name="OrangePLA"/>
+    </visual>
+    <collision>
+        <origin xyz="-0.0455 -0.0415 0" rpy="0 0 0"/>
+        <geometry>
+        <mesh filename="package://eezybot_mk2_description/meshes/EBAmk2_013_lower_base.STL"
+            scale="0.001 0.001 0.001"/>
+        </geometry>
+    </collision>
+    <inertial>
+        <origin xyz="0 0 0"/>
+        <mass value="0.0053"/>
+        <inertia ixx="0.001" ixy="0.0" ixz="0.0"
+                iyy="0.001" iyz="0.0"
+                izz="0.001"/>
+    </inertial>
+    </link>
+    <joint name="lower_base_joint" type="fixed">
+        <parent link="main_base"/>
+        <child link="lower_base"/>
+        <origin xyz="0.06 0 0.03" rpy="0 0 0"/>
+    </joint>
+    <link name="gear_mast">
+    <visual>
+        <origin xyz="-0.039 0.039 0" rpy="${pi} 0 0"/>
+        <geometry>
+        <mesh filename="package://eezybot_mk2_description/meshes/EBAmk2_011_gearmast_full.STL"
+            scale="0.001 0.001 0.001"/>
+        </geometry>
+        <material name="OrangePLA"/>
+    </visual>
+    <collision>
+        <origin xyz="-0.039 0.039 0" rpy="${pi} 0 0"/>
+        <geometry>
+        <mesh filename="package://eezybot_mk2_description/meshes/EBAmk2_011_gearmast_full.STL"
+            scale="0.001 0.001 0.001"/>
+        </geometry>
+    </collision>
+    <inertial>
+        <origin xyz="0 0 0"/>
+        <mass value="0.0053"/>
+        <inertia ixx="0.001" ixy="0.0" ixz="0.0"
+                iyy="0.001" iyz="0.0"
+                izz="0.001"/>
+    </inertial>
+    </link>
+    <joint name="gear_mast_joint" type="revolute">
+        <parent link="lower_base"/>
+        <child link="gear_mast"/>
+        <origin xyz="0 0 0.019" rpy="0 0 0"/>
+        <axis xyz="0.0 0.0 1.0"/>
+        <limit lower="-1.57" upper="1.57" effort="5.0" velocity="1.0"/>
+        <dynamics damping="0.1" friction="0.01"/>
+        <safety_controller soft_lower_limit="-1.4" soft_upper_limit="1.4" k_position="10" k_velocity="5"/>
+        <calibration rising="0.0" falling="0.0"/>
+        <mimic joint="MG996r_conn1_joint" multiplier="-1.0" offset="0.0"/>
+    </joint>
+    <link name="upper_base">
+    <visual>
+        <origin xyz="-0.0445 0.0405 0" rpy="0 0 ${-pi/2}"/>
+        <geometry>
+        <mesh filename="package://eezybot_mk2_description/meshes/EBAmk2_001_base.STL"
+            scale="0.001 0.001 0.001"/>
+        </geometry>
+        <material name="OrangePLA"/>
+    </visual>
+    <collision>
+        <origin xyz="-0.0445 0.0405 0" rpy="0 0 ${-pi/2}"/>
+        <geometry>
+        <mesh filename="package://eezybot_mk2_description/meshes/EBAmk2_001_base.STL"
+            scale="0.001 0.001 0.001"/>
+        </geometry>
+    </collision>
+    <inertial>
+        <origin xyz="0 0 0"/>
+        <mass value="0.0053"/>
+        <inertia ixx="0.001" ixy="0.0" ixz="0.0"
+                iyy="0.001" iyz="0.0"
+                izz="0.001"/>
+    </inertial>
+    </link>
+    <joint name="upper_base_joint" type="fixed">
+        <parent link="gear_mast"/>
+        <child link="upper_base"/>
+        <origin xyz="0 0 0" rpy="0 0 0"/>
+    </joint>
 </robot>

File: eezybot_mk2_description/urdf/mk2_materials.urdf.xacro (robot description, xacro)
@@ -1,6 +1,9 @@
 <?xml version="1.0"?>
 <robot xmlns:xacro="http://www.ros.org/wiki/xacro">
-    <material name="SoftBlack">
-        <color rgba="0.2 0.2 0.2 1.0"/>
+    <material name="BlackPLA">
+        <color rgba="0.5 0.5 0.5 1.0"/>
+    </material>
+    <material name="OrangePLA">
+        <color rgba="0.6 0.3 0.0 1.0"/>
     </material>
 </robot>

Commit message: Ezzybot MK2 Description: Added second servo

File: eezybot_mk2_description/urdf/mk2_base.urdf.xacro (robot description, xacro)
@@ -216,3 +216,62 @@
         <origin xyz="0 0 0" rpy="0 0 0"/>
     </joint>
+    <link name="MG996r_2">
+    <visual>
+        <origin xyz="0 0 0" rpy="${-pi/2} ${-pi/2} 0"/>
+        <geometry>
+        <mesh filename="package://eezybot_mk2_description/meshes/MG946R-MG946R.stl"
+            scale="1 1 1"/>
+        </geometry>
+        <material name="BlackPLA"/>
+    </visual>
+    <collision>
+        <origin xyz="0 0 0" rpy="${-pi/2} ${-pi/2} 0"/>
+        <geometry>
+        <mesh filename="package://eezybot_mk2_description/meshes/MG946R-MG946R.stl"
+            scale="1 1 1"/>
+        </geometry>
+    </collision>
+    <inertial>
+        <origin xyz="0 0 0"/>
+        <mass value="0.0053"/>
+        <inertia ixx="0.001" ixy="0.0" ixz="0.0"
+                iyy="0.001" iyz="0.0"
+                izz="0.001"/>
+    </inertial>
+    </link>
+    <joint name="MG996r_2_joint" type="fixed">
+        <parent link="upper_base"/>
+        <child link="MG996r_2"/>
+        <origin xyz="0.002 -0.054 0.0335" rpy="0 0 0"/>
+    </joint>
+    <link name="MG996r_conn2">
+    <visual>
+        <origin xyz="-0.0165 -0.0071 0" rpy="-${pi/2} 0 0"/>
+        <geometry>
+        <mesh filename="package://eezybot_mk2_description/meshes/TG9_HORN.stl"
+            scale="1 1 1"/>
+        </geometry>
+        <material name="BlackPLA"/>
+    </visual>
+    <collision>
+        <origin xyz="-0.0165 -0.007 0" rpy="-${pi/2} 0 0"/>
+        <geometry>
+        <mesh filename="package://eezybot_mk2_description/meshes/TG9_HORN.stl"
+            scale="1 1 1"/>
+        </geometry>
+    </collision>
+    <inertial>
+        <origin xyz="0 0 0"/>
+        <mass value="0.0053"/>
+        <inertia ixx="0.001" ixy="0.0" ixz="0.0"
+                iyy="0.001" iyz="0.0"
+                izz="0.001"/>
+    </inertial>
+    </link>
+    <joint name="MG996r_conn2_joint" type="revolute">
+        <parent link="MG996r_2"/>
+        <child link="MG996r_conn2"/>
+        <limit lower="${-pi/2}" upper="${pi/2}" effort="0.01" velocity="0.01"/>
+        <origin xyz="0 0 0" rpy="0 0 0"/>
+    </joint>
 </robot>

Commit message: Eezybot MK2 Description: Fixing servo rotation and added main arm

File: eezybot_mk2_description/urdf/mk2_base.urdf.xacro (robot description, xacro)
@@ -247,5 +247,5 @@
     <link name="MG996r_conn2">
     <visual>
-        <origin xyz="-0.0165 -0.0071 0" rpy="-${pi/2} 0 0"/>
+        <origin xyz="-0.01675 -0.006 0" rpy="-${pi/2} 0 0"/>
         <geometry>
         <mesh filename="package://eezybot_mk2_description/meshes/TG9_HORN.stl"
@@ -255,5 +255,5 @@
     </visual>
     <collision>
-        <origin xyz="-0.0165 -0.007 0" rpy="-${pi/2} 0 0"/>
+        <origin xyz="-0.01675 -0.006 0" rpy="-${pi/2} 0 0"/>
         <geometry>
         <mesh filename="package://eezybot_mk2_description/meshes/TG9_HORN.stl"
@@ -272,6 +272,36 @@
         <parent link="MG996r_2"/>
         <child link="MG996r_conn2"/>
+        <axis xyz="0.0 0.0 1.0"/>
         <limit lower="${-pi/2}" upper="${pi/2}" effort="0.01" velocity="0.01"/>
-        <origin xyz="0 0 0" rpy="0 0 0"/>
+        <origin xyz="0 0.0335 0.0095" rpy="${-pi/2} ${-pi/2} 0"/>
+    </joint>
+    <link name="main_arm">
+    <visual>
+        <origin xyz="-0.0195 -0.0120 0.0175" rpy="0 ${pi} ${-pi/2 - 0.225}"/>
+        <geometry>
+        <mesh filename="package://eezybot_mk2_description/meshes/EBAmk2_002_mainarm.STL"
+            scale="0.001 0.001 0.001"/>
+        </geometry>
+        <material name="OrangePLA"/>
+    </visual>
+    <collision>
+        <origin xyz="-0.0195 -0.0120 0.0175" rpy="0 ${pi} ${-pi/2 - 0.225}"/>
+        <geometry>
+        <mesh filename="package://eezybot_mk2_description/meshes/EBAmk2_002_mainarm.STL"
+            scale="0.001 0.001 0.001"/>
+        </geometry>
+    </collision>
+    <inertial>
+        <origin xyz="0 0 0"/>
+        <mass value="0.0053"/>
+        <inertia ixx="0.001" ixy="0.0" ixz="0.0"
+                iyy="0.001" iyz="0.0"
+                izz="0.001"/>
+    </inertial>
+    </link>
+    <joint name="main_arm_joint" type="fixed">
+        <parent link="MG996r_conn2"/>
+        <child link="main_arm"/>
+        <origin xyz="0 0 0.015" rpy="0 0 0"/>
     </joint>
 </robot>

Commit message: Eezybot MK2 Description: Added third servo

File: eezybot_mk2_description/urdf/mk2_base.urdf.xacro (robot description, xacro)
@@ -1,5 +1,7 @@
 <?xml version="1.0"?>
 <robot xmlns:xacro="http://www.ros.org/wiki/xacro">
+    <!-- ///////////////////// BASE LINK ////////////////////////////////// -->
     <link name="base_link" />
+    <!-- ///////////////////// MAIN BASE ////////////////////////////////// -->
     <link name="main_base">
     <visual>
@@ -31,4 +33,5 @@
         <origin xyz="0 0 0" rpy="0 0 0"/>
     </joint>
+    <!-- ///////////////////// SERVO #1 ////////////////////////////////// -->
     <link name="MG996r_1">
     <visual>
@@ -60,4 +63,5 @@
         <origin xyz="-0.0075 0.001 0.008" rpy="0 0 0"/>
     </joint>
+    <!-- ///////////////////// SERVO CONN 1 /////////////////////////////// -->
     <link name="MG996r_conn1">
     <visual>
@@ -94,4 +98,5 @@
         <calibration rising="0.0" falling="0.0"/>
     </joint>
+    <!-- ///////////////////// GEAR SERVO 1 /////////////////////////////// -->
     <link name="gearservo_1">
     <visual>
@@ -123,4 +128,5 @@
         <origin xyz="0 0 0.0025" rpy="0 0 0"/>
     </joint>
+    <!-- ///////////////////// LOWER BASE ////////////////////////////////// -->
     <link name="lower_base">
     <visual>
@@ -152,4 +158,5 @@
         <origin xyz="0.06 0 0.03" rpy="0 0 0"/>
     </joint>
+    <!-- ///////////////////// GEAR BASE ////////////////////////////////// -->
     <link name="gear_mast">
     <visual>
@@ -187,4 +194,5 @@
         <mimic joint="MG996r_conn1_joint" multiplier="-1.0" offset="0.0"/>
     </joint>
+    <!-- ///////////////////// UPPER BASE //////////////////////////////// -->
     <link name="upper_base">
     <visual>
@@ -216,4 +224,5 @@
         <origin xyz="0 0 0" rpy="0 0 0"/>
     </joint>
+    <!-- //////////////////////// SERVO 2 ////////////////////////////////// -->
     <link name="MG996r_2">
     <visual>
@@ -245,4 +254,5 @@
         <origin xyz="0.002 -0.054 0.0335" rpy="0 0 0"/>
     </joint>
+    <!-- ///////////////////// SERVO CONN 2 ////////////////////////////////// -->
     <link name="MG996r_conn2">
     <visual>
@@ -276,4 +286,5 @@
         <origin xyz="0 0.0335 0.0095" rpy="${-pi/2} ${-pi/2} 0"/>
     </joint>
+    <!-- ////////////////////// MAIN ARM ////////////////////////////////// -->
     <link name="main_arm">
     <visual>
@@ -305,3 +316,95 @@
         <origin xyz="0 0 0.015" rpy="0 0 0"/>
     </joint>
+    <!-- /////////////////////// SERVO 3 ////////////////////////////////// -->
+    <link name="MG996r_3">
+    <visual>
+        <origin xyz="0 0 0" rpy="${pi/2} ${-pi/2} 0"/>
+        <geometry>
+        <mesh filename="package://eezybot_mk2_description/meshes/MG946R-MG946R.stl"
+            scale="1 1 1"/>
+        </geometry>
+        <material name="BlackPLA"/>
+    </visual>
+    <collision>
+        <origin xyz="0 0 0" rpy="${pi/2} ${-pi/2} 0"/>
+        <geometry>
+        <mesh filename="package://eezybot_mk2_description/meshes/MG946R-MG946R.stl"
+            scale="1 1 1"/>
+        </geometry>
+    </collision>
+    <inertial>
+        <origin xyz="0 0 0"/>
+        <mass value="0.0053"/>
+        <inertia ixx="0.001" ixy="0.0" ixz="0.0"
+                iyy="0.001" iyz="0.0"
+                izz="0.001"/>
+    </inertial>
+    </link>
+    <joint name="MG996r_3_joint" type="fixed">
+        <parent link="upper_base"/>
+        <child link="MG996r_3"/>
+        <origin xyz="0.002 0.055 0.0335" rpy="0 0 0"/>
+    </joint>
+    <!-- ///////////////////// SERVO CONN 3 /////////////////////////////// -->
+    <link name="MG996r_conn3">
+    <visual>
+        <origin xyz="-0.01675 -0.006 0" rpy="-${pi/2} 0 0"/>
+        <geometry>
+        <mesh filename="package://eezybot_mk2_description/meshes/TG9_HORN.stl"
+            scale="1 1 1"/>
+        </geometry>
+        <material name="BlackPLA"/>
+    </visual>
+    <collision>
+        <origin xyz="-0.01675 -0.006 0" rpy="-${pi/2} 0 0"/>
+        <geometry>
+        <mesh filename="package://eezybot_mk2_description/meshes/TG9_HORN.stl"
+            scale="1 1 1"/>
+        </geometry>
+    </collision>
+    <inertial>
+        <origin xyz="0 0 0"/>
+        <mass value="0.0053"/>
+        <inertia ixx="0.001" ixy="0.0" ixz="0.0"
+                iyy="0.001" iyz="0.0"
+                izz="0.001"/>
+    </inertial>
+    </link>
+    <joint name="MG996r_conn3_joint" type="revolute">
+        <parent link="MG996r_3"/>
+        <child link="MG996r_conn3"/>
+        <axis xyz="0.0 0.0 1.0"/>
+        <limit lower="${-pi}" upper="${0}" effort="0.01" velocity="0.01"/>
+        <origin xyz="0 -0.0335 0.0095" rpy="${pi/2} ${pi} 0"/>
+    </joint>
+    <!-- //////////////////////// V ARM ////////////////////////////////// -->
+    <link name="v_arm">
+    <visual>
+        <origin xyz="-0.015 0.015 0" rpy="${pi} 0 0"/>
+        <geometry>
+        <mesh filename="package://eezybot_mk2_description/meshes/EBAmk2_003_varm.STL"
+            scale="0.001 0.001 0.001"/>
+        </geometry>
+        <material name="OrangePLA"/>
+    </visual>
+    <collision>
+        <origin xyz="-0.015 0.015 0" rpy="${pi} 0 0"/>
+        <geometry>
+        <mesh filename="package://eezybot_mk2_description/meshes/EBAmk2_003_varm.STL"
+            scale="0.001 0.001 0.001"/>
+        </geometry>
+    </collision>
+    <inertial>
+        <origin xyz="0 0 0"/>
+        <mass value="0.0053"/>
+        <inertia ixx="0.001" ixy="0.0" ixz="0.0"
+                iyy="0.001" iyz="0.0"
+                izz="0.001"/>
+    </inertial>
+    </link>
+    <joint name="v_arm_joint" type="fixed">
+        <parent link="MG996r_conn3"/>
+        <child link="v_arm"/>
+        <origin xyz="0 0 0.01" rpy="0 0 0"/>
+    </joint>
 </robot>

Commit message: Eezybot MK2 Description: Added link 135 and horarm, pending fixing orientation

File: eezybot_mk2_description/urdf/mk2_base.urdf.xacro (robot description, xacro)
@@ -408,3 +408,69 @@
         <origin xyz="0 0 0.01" rpy="0 0 0"/>
     </joint>
+    <!-- ///////////////////////// HORARM ////////////////////////////////// -->
+    <link name="hor_arm">
+    <visual>
+        <origin xyz="0.0305 0.153 0" rpy=" ${pi} ${pi/2} 0"/>
+        <geometry>
+        <mesh filename="package://eezybot_mk2_description/meshes/EBAmk2_006_horarm__.STL"
+            scale="0.001 0.001 0.001"/>
+        </geometry>
+        <material name="OrangePLA"/>
+    </visual>
+    <collision>
+        <origin xyz="0.0305 0.153 0" rpy=" ${pi} ${pi/2} 0"/>
+        <geometry>
+        <mesh filename="package://eezybot_mk2_description/meshes/EBAmk2_006_horarm__.STL"
+            scale="0.001 0.001 0.001"/>
+        </geometry>
+    </collision>
+    <inertial>
+        <origin xyz="0 0 0"/>
+        <mass value="0.0053"/>
+        <inertia ixx="0.001" ixy="0.0" ixz="0.0"
+                iyy="0.001" iyz="0.0"
+                izz="0.001"/>
+    </inertial>
+    </link>
+    <joint name="hor_arm_joint" type="revolute">
+        <parent link="main_arm"/>
+        <child link="hor_arm"/>
+        <axis xyz="0.0 0.0 1.0"/>
+        <limit lower="${-pi}" upper="${0}" effort="0.01" velocity="0.01"/>
+        <origin xyz="0.132 -0.03 0.02575" rpy="0 0 0"/>
+        <mimic joint="MG996r_conn3_joint" multiplier="-1.0" offset="0.0"/>
+    </joint>
+    <!-- ///////////////////////// LINK135 ////////////////////////////////// -->
+    <link name="link135_arm">
+    <visual>
+        <origin xyz="-0.00675 0.00675 0" rpy="0 ${pi} ${pi}"/>
+        <geometry>
+        <mesh filename="package://eezybot_mk2_description/meshes/EBAmk2_004_link135.STL"
+            scale="0.001 0.001 0.001"/>
+        </geometry>
+        <material name="OrangePLA"/>
+    </visual>
+    <collision>
+        <origin xyz="-0.00675 0.00675 0" rpy="0 ${pi} ${pi}"/>
+        <geometry>
+        <mesh filename="package://eezybot_mk2_description/meshes/EBAmk2_004_link135.STL"
+            scale="0.001 0.001 0.001"/>
+        </geometry>
+    </collision>
+    <inertial>
+        <origin xyz="0 0 0"/>
+        <mass value="0.0053"/>
+        <inertia ixx="0.001" ixy="0.0" ixz="0.0"
+                iyy="0.001" iyz="0.0"
+                izz="0.001"/>
+    </inertial>
+    </link>
+    <joint name="link135_arm_joint" type="revolute">
+        <parent link="v_arm"/>
+        <child link="link135_arm"/>
+        <axis xyz="0.0 0.0 1.0"/>
+        <limit lower="${-pi/2}" upper="${pi/2}" effort="0.01" velocity="0.01"/>
+        <origin xyz="0.055 0 -0.005" rpy="0 0 ${pi/12}"/>
+        <mimic joint="MG996r_conn2_joint" multiplier="-1.5" offset="0.0"/>
+    </joint>
 </robot>
