Commit message: Description: Adding gripper | GZ: Adding launch with clock

File: eezybot_mk2_description/urdf/mk2.urdf.xacro (robot description, xacro)
@@ -1,7 +1,9 @@
 <?xml version="1.0"?>
 <robot xmlns:xacro="http://www.ros.org/wiki/xacro" name="eezybot_mk2">
+    <xacro:property name="extras" value="false"/>
     <!-- Include other files -->
     <xacro:include filename="$(find eezybot_mk2_description)/urdf/mk2_materials.urdf.xacro"/>
     <xacro:include filename="$(find eezybot_mk2_description)/urdf/mk2_base.urdf.xacro"/>
     <xacro:include filename="$(find eezybot_mk2_description)/urdf/mk2_sim.urdf.xacro"/>
+    <xacro:include filename="$(find eezybot_mk2_description)/urdf/mk2_gazebo.urdf.xacro"/>
 </robot>

File: eezybot_mk2_description/urdf/mk2_base.urdf.xacro (robot description, xacro)
@@ -441,37 +441,39 @@
         <mimic joint="MG996r_conn3_joint" multiplier="-1.0" offset="0.0"/>
     </joint>
-    <!-- ///////////////////////// LINK135 ////////////////////////////////// -->
-    <link name="link135_arm">
-    <visual>
-        <origin xyz="-0.00675 0.00675 0" rpy="0 ${pi} ${pi}"/>
-        <geometry>
-        <mesh filename="package://eezybot_mk2_description/meshes/EBAmk2_004_link135.STL"
-            scale="0.001 0.001 0.001"/>
-        </geometry>
-        <material name="OrangePLA"/>
-    </visual>
-    <collision>
-        <origin xyz="-0.00675 0.00675 0" rpy="0 ${pi} ${pi}"/>
-        <geometry>
-        <mesh filename="package://eezybot_mk2_description/meshes/EBAmk2_004_link135.STL"
-            scale="0.001 0.001 0.001"/>
-        </geometry>
-    </collision>
-    <inertial>
-        <origin xyz="0 0 0"/>
-        <mass value="0.0053"/>
-        <inertia ixx="0.001" ixy="0.0" ixz="0.0"
-                iyy="0.001" iyz="0.0"
-                izz="0.001"/>
-    </inertial>
-    </link>
-    <joint name="link135_arm_joint" type="revolute">
-        <parent link="v_arm"/>
-        <child link="link135_arm"/>
-        <axis xyz="0.0 0.0 1.0"/>
-        <limit lower="${-pi/2}" upper="${pi/2}" effort="0.01" velocity="0.01"/>
-        <origin xyz="0.055 0 -0.005" rpy="0 0 ${pi/12}"/>
-        <mimic joint="MG996r_conn2_joint" multiplier="-1.5" offset="0.0"/>
-    </joint>
+    <xacro:if value="${extras}">
+        <!-- ///////////////////////// LINK135 ////////////////////////////////// -->
+        <link name="link135_arm">
+            <visual>
+                <origin xyz="-0.00675 0.00675 0" rpy="0 ${pi} ${pi}"/>
+                <geometry>
+                    <mesh filename="package://eezybot_mk2_description/meshes/EBAmk2_004_link135.STL"
+                    scale="0.001 0.001 0.001"/>
+                </geometry>
+                <material name="OrangePLA"/>
+            </visual>
+            <collision>
+                <origin xyz="-0.00675 0.00675 0" rpy="0 ${pi} ${pi}"/>
+                <geometry>
+                    <mesh filename="package://eezybot_mk2_description/meshes/EBAmk2_004_link135.STL"
+                    scale="0.001 0.001 0.001"/>
+                </geometry>
+            </collision>
+            <inertial>
+                <origin xyz="0 0 0"/>
+                <mass value="0.0053"/>
+                <inertia ixx="0.001" ixy="0.0" ixz="0.0"
+                iyy="0.001" iyz="0.0"
+                izz="0.001"/>
+            </inertial>
+        </link>
+        <joint name="link135_arm_joint" type="revolute">
+            <parent link="v_arm"/>
+            <child link="link135_arm"/>
+            <axis xyz="0.0 0.0 1.0"/>
+            <limit lower="${-pi/2}" upper="${pi/2}" effort="0.01" velocity="0.01"/>
+            <origin xyz="0.055 0 -0.005" rpy="0 0 ${pi/12}"/>
+            <mimic joint="MG996r_conn2_joint" multiplier="-1.5" offset="0.0"/>
+        </joint>
+    </xacro:if>
     <!-- ///////////////////////// TRIALINK ////////////////////////////////// -->
     <link name="tria_link">
@@ -567,5 +569,5 @@
     <link name="sg90_conn">
     <visual>
-        <origin xyz="-0.01675 -0.006 0" rpy="-${pi/2} 0 0"/>
+        <origin xyz="0.006 -0.01675 0" rpy="-${pi/2} 0 ${pi/2}"/>
         <geometry>
         <mesh filename="package://eezybot_mk2_description/meshes/TG9_HORN.stl"
@@ -575,5 +577,5 @@
     </visual>
     <collision>
-        <origin xyz="-0.01675 -0.006 0" rpy="-${pi/2} 0 0"/>
+        <origin xyz="0.006 -0.01675 0" rpy="-${pi/2} 0 ${pi/2}"/>
         <geometry>
         <mesh filename="package://eezybot_mk2_description/meshes/TG9_HORN.stl"
@@ -593,11 +595,11 @@
         <child link="sg90_conn"/>
         <axis xyz="0.0 0.0 1.0"/>
-        <limit lower="${0}" upper="${pi}" effort="1.0" velocity="1.0"/>
-        <origin xyz="-0.0035 0.005 0" rpy="0 ${-pi/2} 0"/>
+        <limit lower="${0}" upper="${pi/2}" effort="1.0" velocity="1.0"/>
+        <origin xyz="-0.005 0.005 0" rpy="0 ${-pi/2} 0"/>
     </joint>
     <!-- /////////////////////// FIRST GEAR ////////////////////////////////// -->
     <link name="first_gear">
     <visual>
-        <origin xyz="-0.009 0.009 0" rpy="${pi} 0 0"/>
+        <origin xyz="0.0065 -0.0105 0" rpy="0 0 ${pi/2 - pi/12}"/>
         <geometry>
         <mesh filename="package://eezybot_mk2_description/meshes/EBAmk2_016_claw_gear_drive.STL"
@@ -607,5 +609,5 @@
     </visual>
     <collision>
-        <origin xyz="-0.009 0.009 0" rpy="${pi} 0 0"/>
+        <origin xyz="0.065 -0.0105 0" rpy="0 0 ${pi/2 - pi/12}"/>
         <geometry>
         <mesh filename="package://eezybot_mk2_description/meshes/EBAmk2_016_claw_gear_drive.STL"
@@ -624,10 +626,10 @@
         <parent link="sg90_conn"/>
         <child link="first_gear"/>
-        <origin xyz="0 0 0.0055" rpy="0 0 ${pi/12}"/>
-    </joint>
-    <!-- /////////////////////// SEC GEAR ////////////////////////////////// -->
+        <origin xyz="0 0 0" rpy="0 0 0"/>
+    </joint>
+    <!-- /////////////////////// SEC GEAR //////////////////////////////////-->
     <link name="sec_gear">
     <visual>
-        <origin xyz="0 0 0" rpy="${pi} 0 0"/>
+        <origin xyz="0.0075 0.0125 0" rpy="${pi} 0 ${-pi/2}"/>
         <geometry>
         <mesh filename="package://eezybot_mk2_description/meshes/EBAmk2_018_claw_gear_driven.STL"
@@ -637,5 +639,5 @@
     </visual>
     <collision>
-        <origin xyz="0 0 0" rpy="${pi} 0 0"/>
+        <origin xyz="0.0075 0.0125 0" rpy="${pi} 0 ${-pi/2}"/>
         <geometry>
         <mesh filename="package://eezybot_mk2_description/meshes/EBAmk2_018_claw_gear_driven.STL"
@@ -654,8 +656,71 @@
         <parent link="sg90"/>
         <child link="sec_gear"/>
-        <origin xyz="-0.0025 -0.0135 0.0055" rpy="0 ${-pi/2} 0"/>
+        <origin xyz="-0.0095 -0.01225 0.009" rpy="0 ${-pi/2} 0"/>
         <axis xyz="0.0 0.0 1.0"/>
         <limit lower="-1.57" upper="1.57" effort="5.0" velocity="1.0"/>
-        <mimic joint="sg90_conn_joint" multiplier="-1.0" offset="0.0"/>
+        <mimic joint="sg90_conn_joint" multiplier="-0.5" offset="0.0"/>
+    </joint>
+    <!-- /////////////////////// LEFT GRIPPER //////////////////////////////////-->
+    <link name="left_gripper">
+        <visual>
+            <origin xyz="-0.0015 0.049 0" rpy="${pi} 0 ${-pi/2 + pi/12}"/>
+            <geometry>
+            <mesh filename="package://eezybot_mk2_description/meshes/EBAmk2_017_claw_finger_sx.STL"
+                scale="0.001 0.001 0.001"/>
+            </geometry>
+            <material name="OrangePLA"/>
+        </visual>
+        <collision>
+            <origin xyz="-0.0015 0.049 0" rpy="${pi} 0 ${-pi/2 + pi/12}"/>
+            <geometry>
+            <mesh filename="package://eezybot_mk2_description/meshes/EBAmk2_017_claw_finger_sx.STL"
+                scale="0.001 0.001 0.001"/>
+            </geometry>
+        </collision>
+        <inertial>
+            <origin xyz="0 0 0"/>
+            <mass value="0.0053"/>
+            <inertia ixx="0.001" ixy="0.0" ixz="0.0"
+                    iyy="0.001" iyz="0.0"
+                    izz="0.001"/>
+        </inertial>
+    </link>
+    <joint name="left_gripper_joint" type="fixed">
+        <parent link="sec_gear"/>
+        <child link="left_gripper"/>
+        <origin xyz="0 0 -0.00575" rpy="0 0 0"/>
+    </joint>
+    <!-- /////////////////////// RIGHT GRIPPER //////////////////////////////////-->
+    <link name="right_gripper">
+        <visual>
+            <origin xyz="0.01 0.047 0" rpy="${pi} 0 ${-pi/2}"/>
+            <geometry>
+            <mesh filename="package://eezybot_mk2_description/meshes/EBAmk2_015_claw_finger_dx.STL"
+                scale="0.001 0.001 0.001"/>
+            </geometry>
+            <material name="OrangePLA"/>
+        </visual>
+        <collision>
+            <origin xyz="0.01 0.047 0" rpy="${pi} 0 ${-pi/2}"/>
+            <geometry>
+            <mesh filename="package://eezybot_mk2_description/meshes/EBAmk2_015_claw_finger_dx.STL"
+                scale="0.001 0.001 0.001"/>
+            </geometry>
+        </collision>
+        <inertial>
+            <origin xyz="0 0 0"/>
+            <mass value="0.0053"/>
+            <inertia ixx="0.001" ixy="0.0" ixz="0.0"
+                    iyy="0.001" iyz="0.0"
+                    izz="0.001"/>
+        </inertial>
+    </link>
+    <joint name="right_gripper_joint" type="revolute">
+        <parent link="sg90"/>
+        <child link="right_gripper"/>
+        <origin xyz="-0.004 -0.01225 -0.009" rpy="0 ${-pi/2} 0"/>
+        <axis xyz="0.0 0.0 1.0"/>
+        <limit lower="-1.57" upper="1.57" effort="5.0" velocity="1.0"/>
+        <mimic joint="sec_gear_joint" multiplier="-1.0" offset="0.0"/>
     </joint>
 </robot>
