Commit message: Description: Changed limits for joints | GZ: First integration of Joint Position Controllers

File: eezybot_mk2_description/urdf/include/mk2_base.urdf.xacro (robot description, xacro)
@@ -283,5 +283,5 @@
         <child link="MG996r_conn2"/>
         <axis xyz="0.0 0.0 1.0"/>
-        <limit lower="${-pi/2}" upper="${pi/2}" effort="0.01" velocity="0.01"/>
+        <limit lower="${-pi/6}" upper="${pi/4}" effort="0.01" velocity="0.01"/>
         <origin xyz="0 0.0335 0.0095" rpy="${-pi/2} ${-pi/2} 0"/>
     </joint>
@@ -376,36 +376,39 @@
         <axis xyz="0.0 0.0 1.0"/>
         <limit lower="${-pi}" upper="${0}" effort="0.01" velocity="0.01"/>
+        <mimic joint="hor_arm_joint" multiplier="-1.0" offset="0.0"/>
         <origin xyz="0 -0.0335 0.0095" rpy="${pi/2} ${pi} 0"/>
     </joint>
-    <!-- //////////////////////// V ARM ////////////////////////////////// -->
-    <link name="v_arm">
-    <visual>
-        <origin xyz="-0.015 0.015 0" rpy="${pi} 0 0"/>
-        <geometry>
-        <mesh filename="package://eezybot_mk2_description/meshes/EBAmk2_003_varm.STL"
-            scale="0.001 0.001 0.001"/>
-        </geometry>
-        <material name="OrangePLA"/>
-    </visual>
-    <collision>
-        <origin xyz="-0.015 0.015 0" rpy="${pi} 0 0"/>
-        <geometry>
-        <mesh filename="package://eezybot_mk2_description/meshes/EBAmk2_003_varm.STL"
-            scale="0.001 0.001 0.001"/>
-        </geometry>
-    </collision>
-    <inertial>
-        <origin xyz="0 0 0"/>
-        <mass value="0.0053"/>
-        <inertia ixx="0.001" ixy="0.0" ixz="0.0"
-                iyy="0.001" iyz="0.0"
-                izz="0.001"/>
-    </inertial>
-    </link>
-    <joint name="v_arm_joint" type="fixed">
-        <parent link="MG996r_conn3"/>
-        <child link="v_arm"/>
-        <origin xyz="0 0 0.01" rpy="0 0 0"/>
-    </joint>
+    <xacro:if value="${extras}">
+        <!-- //////////////////////// V ARM ////////////////////////////////// -->
+        <link name="v_arm">
+        <visual>
+            <origin xyz="-0.015 0.015 0" rpy="${pi} 0 0"/>
+            <geometry>
+            <mesh filename="package://eezybot_mk2_description/meshes/EBAmk2_003_varm.STL"
+                scale="0.001 0.001 0.001"/>
+            </geometry>
+            <material name="OrangePLA"/>
+        </visual>
+        <collision>
+            <origin xyz="-0.015 0.015 0" rpy="${pi} 0 0"/>
+            <geometry>
+            <mesh filename="package://eezybot_mk2_description/meshes/EBAmk2_003_varm.STL"
+                scale="0.001 0.001 0.001"/>
+            </geometry>
+        </collision>
+        <inertial>
+            <origin xyz="0 0 0"/>
+            <mass value="0.0053"/>
+            <inertia ixx="0.001" ixy="0.0" ixz="0.0"
+                    iyy="0.001" iyz="0.0"
+                    izz="0.001"/>
+        </inertial>
+        </link>
+        <joint name="v_arm_joint" type="fixed">
+            <parent link="MG996r_conn3"/>
+            <child link="v_arm"/>
+            <origin xyz="0 0 0.01" rpy="0 0 0"/>
+        </joint>
+    </xacro:if>
     <!-- ///////////////////////// HORARM ////////////////////////////////// -->
     <link name="hor_arm">
@@ -437,7 +440,6 @@
         <child link="hor_arm"/>
         <axis xyz="0.0 0.0 1.0"/>
-        <limit lower="${-pi}" upper="${0}" effort="0.01" velocity="0.01"/>
+        <limit lower="${-pi/8}" upper="${pi/4}" effort="0.01" velocity="0.01"/>
         <origin xyz="0.132 -0.03 0.02575" rpy="0 0 0"/>
-        <mimic joint="MG996r_conn3_joint" multiplier="-1.0" offset="0.0"/>
     </joint>
     <xacro:if value="${extras}">

File: eezybot_mk2_gz/urdf/include/mk2_actuators.urdf.xacro (robot description, xacro)
@@ -1,7 +1,65 @@
 <?xml version="1.0"?>
 <robot xmlns:xacro="http://www.ros.org/wiki/xacro">
-    <plugin
-        filename="gz-sim-joint-state-publisher-system"
-        name="gz::sim::systems::JointStatePublisher">
-    </plugin>
+    <gazebo>
+        <plugin
+            filename="gz-sim-joint-position-controller-system"
+            name="gz::sim::systems::JointPositionController">
+            <joint_name>MG996r_conn1_joint</joint_name>
+            <p_gain>10</p_gain>
+            <i_gain>0.1</i_gain>
+            <d_gain>0.01</d_gain>
+            <i_max>1</i_max>
+            <i_min>-1</i_min>
+            <cmd_max>1000</cmd_max>
+            <cmd_min>-1000</cmd_min>
+        </plugin>
+    </gazebo>
+    <gazebo>
+        <plugin
+            filename="gz-sim-joint-position-controller-system"
+            name="gz::sim::systems::JointPositionController">
+            <joint_name>MG996r_conn2_joint</joint_name>
+            <p_gain>10</p_gain>
+            <i_gain>0.1</i_gain>
+            <d_gain>0.01</d_gain>
+            <i_max>1</i_max>
+            <i_min>-1</i_min>
+            <cmd_max>1000</cmd_max>
+            <cmd_min>-1000</cmd_min>
+        </plugin>
+    </gazebo>
+    <gazebo>
+        <plugin
+            filename="gz-sim-joint-position-controller-system"
+            name="gz::sim::systems::JointPositionController">
+            <joint_name>hor_arm_joint</joint_name>
+            <p_gain>10</p_gain>
+            <i_gain>0.1</i_gain>
+            <d_gain>0.01</d_gain>
+            <i_max>1</i_max>
+            <i_min>-1</i_min>
+            <cmd_max>1000</cmd_max>
+            <cmd_min>-1000</cmd_min>
+        </plugin>
+    </gazebo>
+    <gazebo>
+        <plugin
+            filename="gz-sim-joint-position-controller-system"
+            name="gz::sim::systems::JointPositionController">
+            <joint_name>sg90_conn_joint</joint_name>
+            <p_gain>10</p_gain>
+            <i_gain>0.1</i_gain>
+            <d_gain>0.01</d_gain>
+            <i_max>1</i_max>
+            <i_min>-1</i_min>
+            <cmd_max>1000</cmd_max>
+            <cmd_min>-1000</cmd_min>
+        </plugin>
+    </gazebo>
+    <gazebo>
+        <plugin
+            filename="gz-sim-joint-state-publisher-system"
+            name="gz::sim::systems::JointStatePublisher">
+        </plugin>
+    </gazebo>
 </robot>

File: eezybot_mk2_gz/urdf/mk2_gz.urdf.xacro (robot description, xacro)
@@ -6,3 +6,4 @@
     <xacro:include filename="$(find eezybot_mk2_description)/urdf/include/mk2_base.urdf.xacro"/>
     <xacro:include filename="$(find eezybot_mk2_gz)/urdf/include/mk2_gazebo.urdf.xacro"/>
+    <xacro:include filename="$(find eezybot_mk2_gz)/urdf/include/mk2_actuators.urdf.xacro"/>
 </robot>
