Commit message: brazo parcialmente completado urdfs

File: eezybot_mk1_description/urdf/mk1_base.urdf.xacro (robot description, xacro)
@@ -2,4 +2,5 @@
 <robot xmlns:xacro="http://www.ros.org/wiki/xacro">
     <link name="base_link"/>
+    <!--  raund plate , base -->
     <link name="main_base">
     <visual>
@@ -9,5 +10,5 @@
             scale="0.001 0.001 0.001"/>
         </geometry>
-        <color rgba="11 7 75 1.0"/>
+        <material name="sky_blue"/>
     </visual>
     <collision>
@@ -39,5 +40,5 @@
             scale="0.001 0.001 0.001"/>
         </geometry>
-        <color rgba="0.2 0.2 0.2 1.0"/>
+       <material name="sky_blue"/>
     </visual>
     <collision>
@@ -60,8 +61,9 @@
         <child link="raund_plate"/>
         <axis xyz="0 0 1"/>
-        <limit effort="1000.0" lower="0.0" upper="360" velocity="1"/>
+        <limit effort="1000.0" lower="0.0" upper="6" velocity="1"/>
         <origin xyz="0 0 0.031" rpy="0 0 0"/>
     </joint>
 <!-- -->
+<!-- tercera pieza -->
      <link name="over_plate">
     <visual>
@@ -71,5 +73,5 @@
             scale="0.001 0.001 0.001"/>
         </geometry>
-        <color rgba="11 7 75 1.0"/>
+        <material name="sky_blue"/>
     </visual>
     <collision>
@@ -93,3 +95,236 @@
         <origin xyz="0 0 0" rpy="0 0 0"/>
     </joint>
+<!--eezybot_mk1_description/meshes/EBA_01.00.004_forward_drive_arm.STL -->
+<!-- antebrazo parte1 -->
+<link name="arm_part">
+    <visual>
+        <origin xyz="0.018 -0.008 0.008" rpy="0 1.5708 1.5708"/>
+        <geometry>
+        <mesh filename="package://eezybot_mk1_description/meshes/EBA_01.00.004_forward_drive_arm.STL"
+            scale="0.001 0.001 0.001"/>
+        </geometry>
+        <material name="sky_blue"/>
+    </visual>
+    <collision>
+        <origin xyz="0.018 -0.008 0.008" rpy="0 1.5708 1.5708"/>
+        <geometry>
+        <mesh filename="package://eezybot_mk1_description/meshes/EBA_01.00.004_forward_drive_arm.STL"
+            scale="0.001 0.001 0.001"/>
+        </geometry>
+    </collision>
+    <inertial>
+        <origin xyz="0 0 0"/>
+        <mass value="0.0053"/>
+        <inertia ixx="0.001" ixy="0.0" ixz="0.0"
+                iyy="0.001" iyz="0.0"
+                izz="0.001"/>
+    </inertial>
+    </link>
+    <joint name="arm_part_joint" type="revolute">
+        <parent link="over_plate"/>
+        <child link="arm_part"/>
+        <axis xyz="1 0 0"/>
+        <limit effort="1000.0" lower="1.6" upper="5.1" velocity="1"/>
+        <origin xyz="0 0 0.031" rpy="0 0 0"/>
+    </joint>
+<!-- eezybot_mk1_description/meshes/EBA_01.00.002_vertical_drive_arm.STL1.5708-->
+<!-- parte 5_foream_base-->
+<link name="foream_base">
+    <visual>
+        <origin xyz="0.0 0.006 0.04" rpy="3.14 1.5709 0"/>
+        <geometry>
+        <mesh filename="package://eezybot_mk1_description/meshes/EBA_01.00.002_vertical_drive_arm.STL"
+            scale="0.001 0.001 0.001"/>
+        </geometry>
+       <material name="sky_blue"/>
+    </visual>
+    <collision>
+        <origin xyz="0.0 0.006 0.04" rpy="3.14 1.5709 0"/>
+        <geometry>
+        <mesh filename="package://eezybot_mk1_description/meshes/EBA_01.00.002_vertical_drive_arm.STL"
+            scale="0.001 0.001 0.001"/>
+        </geometry>
+    </collision>
+    <inertial>
+        <origin xyz="0 0 0"/>
+        <mass value="0.0053"/>
+        <inertia ixx="0.001" ixy="0.0" ixz="0.0"
+                iyy="0.001" iyz="0.0"
+                izz="0.001"/>
+    </inertial>
+    </link>
+    <joint name="foream_base_joint" type="revolute">
+        <parent link="over_plate"/>
+        <child link="foream_base"/>
+        <axis xyz="1 0 0"/>
+        <limit effort="1000.0" lower="0.0" upper="6" velocity="1"/>
+        <origin xyz="-0.015 0 0.031" rpy="0 0 0"/>
+    </joint>
+<!-- eezybot_mk1_description/meshes/EBA_01.00.005_horizontal_arm.STL-->
+<!-- forearm_part-->
+<link name="forearm_part">
+    <visual>
+        <origin xyz="-0.004 0.043 0.008" rpy="1.5709 3.14 1.5709"/>
+        <geometry>
+        <mesh filename="package://eezybot_mk1_description/meshes/EBA_01.00.005_horizontal_arm.STL"
+            scale="0.001 0.001 0.001"/>
+        </geometry>
+        <material name="sky_blue"/>
+    </visual>
+    <collision>
+        <origin xyz="-0.004 0.043 0.008" rpy="1.5709 3.14 1.5709"/>
+        <geometry>
+        <mesh filename="package://eezybot_mk1_description/meshes/EBA_01.00.005_horizontal_arm.STL"
+            scale="0.001 0.001 0.001"/>
+        </geometry>
+    </collision>
+    <inertial>
+        <origin xyz="0 0 0"/>
+        <mass value="0.0053"/>
+        <inertia ixx="0.001" ixy="0.0" ixz="0.0"
+                iyy="0.001" iyz="0.0"
+                izz="0.001"/>
+    </inertial>
+    </link>
+    <joint name="forearm_part_joint" type="revolute">
+        <parent link="arm_part"/>
+        <child link="forearm_part"/>
+        <axis xyz="1 0 0"/>
+        <limit effort="1000.0" lower="-1.0" upper="6" velocity="1"/>
+        <origin xyz="-0.0 -0.003 -0.08" rpy="0 0 0"/>
+       <!-- <mimic joint= "foream_base_joint" multiplier="1.0" offset="-1.589"/>-->
+    </joint>
+<!-- eezybot_mk1_description/meshes/EBA_01.00.003_link.STL-->
+<!-- Connection_forearm-->
+<link name="Connection_forearm">
+    <visual>
+        <origin xyz="-0.00 -0.006 -0.006" rpy="1.5709 0 1.5709"/>
+        <geometry>
+        <mesh filename="package://eezybot_mk1_description/meshes/EBA_01.00.003_link.STL"
+            scale="0.001 0.001 0.001"/>
+        </geometry>
+        <material name="sky_blue"/>
+    </visual>
+    <collision>
+        <origin xyz="-0.0 -0.006 -0.006" rpy="1.5709 0 1.5709"/>
+        <geometry>
+        <mesh filename="package://eezybot_mk1_description/meshes/EBA_01.00.003_link.STL"
+            scale="0.001 0.001 0.001"/>
+        </geometry>
+    </collision>
+    <inertial>
+        <origin xyz="0 0 0"/>
+        <mass value="0.0053"/>
+        <inertia ixx="0.001" ixy="0.0" ixz="0.0"
+                iyy="0.001" iyz="0.0"
+                izz="0.001"/>
+    </inertial>
+    </link>
+    <joint name="Connection_forearm_joint" type="revolute">
+        <parent link="foream_base"/>
+        <child link="Connection_forearm"/>
+        <axis xyz="1 0 0"/>
+        <limit effort="1000.0" lower="-1.0" upper="6" velocity="1"/>
+        <origin xyz="-0.0 0 0.035" rpy="0 0 0"/>
+    </joint>
+<!--eezybot_mk1_description/meshes/EBA_01.00.012_R01_claw_support.STL-->
+<!-- claw__base-->
+<link name="claw_base">
+    <visual>
+        <origin xyz="0.013 0.0065 0.016" rpy="0 3.14 1.5709"/>
+        <geometry>
+        <mesh filename="package://eezybot_mk1_description/meshes/EBA_01.00.012_R01_claw_support.STL"
+            scale="0.001 0.001 0.001"/>
+        </geometry>
+        <material name="sky_blue"/>
+    </visual>
+    <collision>
+        <origin xyz="0.013 0.0065 0.016" rpy="0 3.14 1.5709"/>
+        <geometry>
+        <mesh filename="package://eezybot_mk1_description/meshes/EBA_01.00.012_R01_claw_support.STL"
+            scale="0.001 0.001 0.001"/>
+        </geometry>
+    </collision>
+    <inertial>
+        <origin xyz="0 0 0"/>
+        <mass value="0.0053"/>
+        <inertia ixx="0.001" ixy="0.0" ixz="0.0"
+                iyy="0.001" iyz="0.0"
+                izz="0.001"/>
+    </inertial>
+    </link>
+    <joint name="claw_base_joint" type="revolute">
+        <parent link="forearm_part"/>
+        <child link="claw_base"/>
+        <axis xyz="1 0 0"/>
+        <origin xyz="-0.0 -0.08 0" rpy="0 0 0"/>
+        <limit effort="1000.0" lower="-1.0" upper="6" velocity="1"/>
+    </joint>
+<!--eezybot_mk1_description/meshes/EBA_01.00.013_R01_right_finger.STL 3.14-->
+<!-- right_finger-->
+<link name="right_finger">
+    <visual>
+        <origin xyz="-0.01 -0.0475 0.004" rpy="3.14 0 1.5709"/>
+        <geometry>
+        <mesh filename="package://eezybot_mk1_description/meshes/EBA_01.00.013_R01_right_finger.STL"
+            scale="0.001 0.001 0.001"/>
+        </geometry>
+        <material name="sky_blue"/>
+    </visual>
+    <collision>
+        <origin xyz="-0.011 -0.047 0.004" rpy="3.14 0 1.5709"/>
+        <geometry>
+        <mesh filename="package://eezybot_mk1_description/meshes/EBA_01.00.013_R01_right_finger.STL"
+            scale="0.001 0.001 0.001"/>
+        </geometry>
+    </collision>
+    <inertial>
+        <origin xyz="0 0 0"/>
+        <mass value="0.0053"/>
+        <inertia ixx="0.001" ixy="0.0" ixz="0.0"
+                iyy="0.001" iyz="0.0"
+                izz="0.001"/>
+    </inertial>
+    </link>
+    <joint name="right_finger_joint" type="revolute">
+        <parent link="claw_base"/>
+        <child link="right_finger"/>
+        <axis xyz="0 0 1"/>
+        <origin xyz="0.009 -0.014 0.016" rpy="0 0 0"/>
+        <limit effort="1000.0" lower="-1.0" upper="6" velocity="1"/>
+    </joint>
+<!--eezybot_mk1_description/meshes/EBA_01.00.014_R01_left_finger.STL-->
+<!-- left_finger-->
+<link name="left_finger">
+    <visual>
+        <origin xyz="-0.0035 -0.0475 0.004" rpy="3.14 0 1.5709"/>
+        <geometry>
+        <mesh filename="package://eezybot_mk1_description/meshes/EBA_01.00.014_R01_left_finger.STL"
+            scale="0.001 0.001 0.001"/>
+        </geometry>
+        <material name="sky_blue"/>
+    </visual>
+    <collision>
+        <origin xyz="-0.011 -0.047 0.004" rpy="3.14 0 1.5709"/>
+        <geometry>
+        <mesh filename="package://eezybot_mk1_description/meshes/EBA_01.00.014_R01_left_finger.STL"
+            scale="0.001 0.001 0.001"/>
+        </geometry>
+    </collision>
+    <inertial>
+        <origin xyz="0 0 0"/>
+        <mass value="0.0053"/>
+        <inertia ixx="0.001" ixy="0.0" ixz="0.0"
+                iyy="0.001" iyz="0.0"
+                izz="0.001"/>
+    </inertial>
+    </link>
+    <joint name="left_finger_joint" type="revolute">
+        <parent link="claw_base"/>
+        <child link="left_finger"/>
+        <axis xyz="0 0 1"/>
+        <origin xyz="-0.009 -0.014 0.016" rpy="0 0 0"/>
+        <limit effort="1000.0" lower="-1.0" upper="6" velocity="1"/>
+        <mimic joint= "right_finger_joint" multiplier="-1.0" offset="-0"/>
+    </joint>
 </robot>

File: eezybot_mk1_description/urdf/mk1_material.urdf.xacro (robot description, xacro)
@@ -5,5 +5,5 @@
     </material>
      <material name="sky_blue">
-        <color rgba="11 7 75 1.0"/>
+        <color rgba="0 0 0 1"/>
     </material>
 </robot>

Commit message: Description: Updating mk1 description

File: eezybot_mk1_description/urdf/mk1_base.urdf.xacro (robot description, xacro)
@@ -20,6 +20,6 @@
     </collision>
     <inertial>
-        <origin xyz="0 0 0"/>
-        <mass value="0.0053"/>
+        <origin xyz="0.029 0.038 0.014"/>
+        <mass value="0.02252"/>
         <inertia ixx="0.001" ixy="0.0" ixz="0.0"
                 iyy="0.001" iyz="0.0"
@@ -158,5 +158,5 @@
         <child link="foream_base"/>
         <axis xyz="1 0 0"/>
-        <limit effort="1000.0" lower="0.0" upper="6" velocity="1"/>
+        <limit effort="1000.0" lower="0.0" upper="2" velocity="1"/>
         <origin xyz="-0.015 0 0.031" rpy="0 0 0"/>
     </joint>
@@ -191,5 +191,5 @@
         <child link="forearm_part"/>
         <axis xyz="1 0 0"/>
-        <limit effort="1000.0" lower="-1.0" upper="6" velocity="1"/>
+        <limit effort="1000.0" lower="-1.0" upper="4" velocity="1"/>
         <origin xyz="-0.0 -0.003 -0.08" rpy="0 0 0"/>
        <!-- <mimic joint= "foream_base_joint" multiplier="1.0" offset="-1.589"/>-->
@@ -225,5 +225,5 @@
         <child link="Connection_forearm"/>
         <axis xyz="1 0 0"/>
-        <limit effort="1000.0" lower="-1.0" upper="6" velocity="1"/>
+        <limit effort="1000.0" lower="-1.0" upper="4" velocity="1"/>
         <origin xyz="-0.0 0 0.035" rpy="0 0 0"/>
     </joint>
@@ -259,5 +259,5 @@
         <axis xyz="1 0 0"/>
         <origin xyz="-0.0 -0.08 0" rpy="0 0 0"/>
-        <limit effort="1000.0" lower="-1.0" upper="6" velocity="1"/>
+        <limit effort="1000.0" lower="-1.0" upper="3" velocity="1"/>
     </joint>
 <!--eezybot_mk1_description/meshes/EBA_01.00.013_R01_right_finger.STL 3.14-->
@@ -273,5 +273,5 @@
     </visual>
     <collision>
-        <origin xyz="-0.011 -0.047 0.004" rpy="3.14 0 1.5709"/>
+        <origin xyz="-0.01 -0.0475 0.004" rpy="3.14 0 1.5709"/>
         <geometry>
         <mesh filename="package://eezybot_mk1_description/meshes/EBA_01.00.013_R01_right_finger.STL"
@@ -292,5 +292,5 @@
         <axis xyz="0 0 1"/>
         <origin xyz="0.009 -0.014 0.016" rpy="0 0 0"/>
-        <limit effort="1000.0" lower="-1.0" upper="6" velocity="1"/>
+        <limit effort="1000.0" lower="0" upper="1.7" velocity="1"/>
     </joint>
 <!--eezybot_mk1_description/meshes/EBA_01.00.014_R01_left_finger.STL-->
@@ -306,5 +306,5 @@
     </visual>
     <collision>
-        <origin xyz="-0.011 -0.047 0.004" rpy="3.14 0 1.5709"/>
+        <origin xyz="-0.0035 -0.0475 0.004" rpy="3.14 0 1.5709"/>
         <geometry>
         <mesh filename="package://eezybot_mk1_description/meshes/EBA_01.00.014_R01_left_finger.STL"
@@ -325,5 +325,5 @@
         <axis xyz="0 0 1"/>
         <origin xyz="-0.009 -0.014 0.016" rpy="0 0 0"/>
-        <limit effort="1000.0" lower="-1.0" upper="6" velocity="1"/>
+        <limit effort="1000.0" lower="-0" upper="1.7" velocity="1"/>
         <mimic joint= "right_finger_joint" multiplier="-1.0" offset="-0"/>
     </joint>

File: eezybot_mk1_description/urdf/mk1_material.urdf.xacro (robot description, xacro)
@@ -5,5 +5,5 @@
     </material>
      <material name="sky_blue">
-        <color rgba="0 0 0 1"/>
+        <color rgba="0.3 0.07 0.7 1"/>
     </material>
 </robot>

File: eezybot_mk1_description/urdf/mk1_sim.urdf.xacro (robot description, xacro)
@@ -1,3 +1,6 @@
 <?xml version="1.0"?>
 <robot xmlns:xacro="http://www.ros.org/wiki/xacro">
+    <gazebo>
+    <plugin filename="ignition-gazebo-joint-state-publisher-system" name="ignition::gazebo::systems::JointStatePublisher"/>
+  </gazebo>
 </robot>
